Commit message: Gazebo world added

File: description/robot.urdf.xacro (robot description, xacro)
@@ -2,3 +2,4 @@
 <robot xmlns:xacro="http://www.ros.org/wiki/xacro"  name="robot">
      <xacro:include filename="robot_core.xacro" />
+     <xacro:include filename="gazebo_control.xacro" />
 </robot>

File: description/robot_core.xacro (robot description, xacro)
@@ -57,4 +57,7 @@
     </xacro:inertial_box>
   </link>
+  <gazebo reference="chassis">
+      <material>Gazebo/White</material>
+  </gazebo>
  <!-- LEFT WHEEL -->
     <joint name="left_wheel_joint" type="continuous">
@@ -63,4 +66,5 @@
         <origin xyz="-0.0675 0.105 0" rpy="-${pi/2} 0 0"/>
         <axis xyz="0 0 1"/>
+        <limit effort="0.05" velocity="10.0"/>
     </joint>
     <link name="left_wheel">
@@ -73,5 +77,6 @@
         <collision>
             <geometry>
-                <cylinder length="0.03" radius="0.033" />
+                <!-- <cylinder length="0.03" radius="0.033" />  -->
+                <sphere radius="0.033" />
             </geometry>
         </collision>
@@ -80,4 +85,7 @@
         </xacro:inertial_cylinder>
     </link>
+    <gazebo reference="left_wheel">
+       <material>Gazebo/Blue</material>
+    </gazebo>
     <!-- RIGHT WHEEL -->
     <joint name="right_wheel_joint" type="continuous">
@@ -86,4 +94,5 @@
         <origin xyz="-0.0675 -0.105 0" rpy="${pi/2} 0 0"/>
         <axis xyz="0 0 -1"/>
+        <limit effort="0.05" velocity="10.0"/>
     </joint>
     <link name="right_wheel">
@@ -96,5 +105,6 @@
         <collision>
             <geometry>
-                <cylinder length="0.03" radius="0.033" />
+                <!-- <cylinder length="0.03" radius="0.033" />  -->
+                <sphere radius="0.033" />
             </geometry>
         </collision>
@@ -103,4 +113,7 @@
         </xacro:inertial_cylinder>
     </link>
+    <gazebo reference="right_wheel">
+       <material>Gazebo/Blue</material>
+    </gazebo>
  <!-- CASTER WHEEL -->
     <joint name="caster_wheel_joint" type="fixed">
@@ -126,3 +139,8 @@
         </xacro:inertial_sphere>
     </link>
+    <gazebo reference="caster_wheel">
+       <material>Gazebo/Black</material>
+        <mu1 value="0.0"/>
+        <mu2 value="0.0"/>
+    </gazebo>
 </robot>

Commit message: Lidar

File: description/robot.urdf.xacro (robot description, xacro)
@@ -3,3 +3,4 @@
      <xacro:include filename="robot_core.xacro" />
      <xacro:include filename="gazebo_control.xacro" />
+      <xacro:include filename="lidar.xacro" />
 </robot>

File: description/robot_core.xacro (robot description, xacro)
@@ -13,4 +13,7 @@
     <material name="black">
         <color rgba="0 0 0 1"/>
+    </material>
+    <material name="red">
+        <color rgba="1 0 0 1"/>
     </material>
    <link name="base_link">
