Commit message: tracking

File: description/robot_core copy.xacro (robot description, xacro)
@@ -31,5 +31,6 @@
         <parent link="base_link"/>
         <child link="chassis"/>
-        <origin xyz="-0.1 0 0"/>
+        <!-- <origin xyz="-0.1 0 0"/> -->
+        <origin xyz="${-wheel_offset_x} 0 ${-wheel_offset_z}"/>
     </joint>
   <link name="chassis">
@@ -76,5 +77,5 @@
         <child link="left_wheel"/>
         <!-- <origin xyz="-0.0675 0.105 0" rpy="-${pi/2} 0 0"/>  -->
-        <origin xyz="-0.10 0.105 0" rpy="-${pi/2} 0 0"/>
+        <origin xyz="-0.0675 0.105 0" rpy="-${pi/2} 0 0"/>
         <axis xyz="0 0 1"/>
         <limit effort="0.05" velocity="10.0"/>
